File: hardware/Microcontroller.sch (KiCad schematic (older format))
At the start: 17 parts, among them J6 AVR-ISP-6, K1 CONN_3, Q1 2N3904, U4 ATMEGA64M1

Commit message: Modified the components in the 3 phase inverter
Parts:
- removed U4: ATMEGA64M1, symbol ATMEGA64C1
- added U4: ATMEGA64M1, symbol ATMEGA64M1
Changed lines of the file:
@@
-EESchema Schematic File Version 2  date Sun 19 Apr 2015 17:21:43 MST
+EESchema Schematic File Version 2  date Sat 25 Apr 2015 16:01:28 MST
 LIBS:power
 LIBS:device
@@
 Sheet 3 4
 Title "Microcontroller and Support"
-Date "19 apr 2015"
+Date "25 apr 2015"
 Rev ""
 Comp ""
@@
 Comment4 ""
 $EndDescr
+$Comp
+L ATMEGA64M1 U4
+U 1 1 553C1091
+P 3800 3650
+F 0 "U4" H 3600 5200 60  0000 C CNN
+F 1 "ATMEGA64M1" H 3800 2100 60  0000 C CNN
+	1    3800 3650
+	1    0    0    -1
+$EndComp
 Wire Wire Line
 	3000 2400 3000 2350
@@
 Connection ~ 3000 2400
 $Comp
-L +5VA #PWR23
+L +5VA #PWR024
 U 1 1 553437E9
 P 3000 2350
-F 0 "#PWR23" H 3000 2480 20  0001 C CNN
+F 0 "#PWR024" H 3000 2480 20  0001 C CNN
 F 1 "+5VA" H 3000 2450 30  0000 C CNN
 	1    3000 2350
@@
 NoConn ~ 4500 2500
 $Comp
-L GND #PWR29
+L GND #PWR025
 U 1 1 553400C3
 P 6950 5200
-F 0 "#PWR29" H 6950 5200 30  0001 C CNN
+F 0 "#PWR025" H 6950 5200 30  0001 C CNN
 F 1 "GND" H 6950 5130 30  0001 C CNN
 	1    6950 5200
@@
 nRESET
 $Comp
-L +5V #PWR31
+L +5V #PWR026
 U 1 1 5533F780
 P 4300 6400
-F 0 "#PWR31" H 4300 6490 20  0001 C CNN
+F 0 "#PWR026" H 4300 6490 20  0001 C CNN
 F 1 "+5V" H 4300 6490 30  0000 C CNN
 	1    4300 6400
@@
 $EndComp
 $Comp
-L GND #PWR32
+L GND #PWR027
 U 1 1 5533F77F
 P 4300 6800
-F 0 "#PWR32" H 4300 6800 30  0001 C CNN
+F 0 "#PWR027" H 4300 6800 30  0001 C CNN
 F 1 "GND" H 4300 6730 30  0001 C CNN
 	1    4300 6800
@@
 $EndComp
 $Comp
-L GND #PWR25
+L GND #PWR028
 U 1 1 5533F766
 P 9250 3200
-F 0 "#PWR25" H 9250 3200 30  0001 C CNN
+F 0 "#PWR028" H 9250 3200 30  0001 C CNN
 F 1 "GND" H 9250 3130 30  0001 C CNN
 	1    9250 3200
@@
 $EndComp
 $Comp
-L +BATT #PWR20
+L +BATT #PWR029
 U 1 1 5533F765
 P 9250 1700
-F 0 "#PWR20" H 9250 1650 20  0001 C CNN
+F 0 "#PWR029" H 9250 1650 20  0001 C CNN
 F 1 "+BATT" H 9250 1800 30  0000 C CNN
 	1    9250 1700
@@
 W_HI
 $Comp
-L ATMEGA64C1 U4
-U 1 1 5533F45D
-P 3800 3650
-F 0 "U4" H 3600 5200 60  0000 C CNN
-F 1 "ATMEGA64M1" H 3800 2100 60  0000 C CNN
-	1    3800 3650
-	1    0    0    -1
-$EndComp
-$Comp
 L INDUCTOR L1
 U 1 1 5533F45C
@@
 $EndComp
 $Comp
-L GND #PWR28
+L GND #PWR030
 U 1 1 5533F45A
 P 3200 5050
-F 0 "#PWR28" H 3200 5050 30  0001 C CNN
+F 0 "#PWR030" H 3200 5050 30  0001 C CNN
 F 1 "GND" H 3200 4980 30  0001 C CNN
 	1    3200 5050
@@
 $EndComp
 $Comp
-L GND #PWR26
+L GND #PWR031
 U 1 1 5533F459
 P 3100 4100
-F 0 "#PWR26" H 3100 4100 30  0001 C CNN
+F 0 "#PWR031" H 3100 4100 30  0001 C CNN
 F 1 "GND" H 3100 4030 30  0001 C CNN
 	1    3100 4100
@@
 $EndComp
 $Comp
-L +5V #PWR21
+L +5V #PWR032
 U 1 1 5533F458
 P 3100 1750
-F 0 "#PWR21" H 3100 1840 20  0001 C CNN
+F 0 "#PWR032" H 3100 1840 20  0001 C CNN
 F 1 "+5V" H 3100 1840 30  0000 C CNN
 	1    3100 1750
@@
 $EndComp
 $Comp
-L GND #PWR24
+L GND #PWR033
 U 1 1 5533F455
 P 3150 2850
-F 0 "#PWR24" H 3150 2850 30  0001 C CNN
+F 0 "#PWR033" H 3150 2850 30  0001 C CNN
 F 1 "GND" H 3150 2780 30  0001 C CNN
 	1    3150 2850
@@
 $EndComp
 $Comp
-L GND #PWR22
+L GND #PWR034
 U 1 1 5533F454
 P 3250 2200
-F 0 "#PWR22" H 3250 2200 30  0001 C CNN
+F 0 "#PWR034" H 3250 2200 30  0001 C CNN
 F 1 "GND" H 3250 2130 30  0001 C CNN
 	1    3250 2200
@@
 $EndComp
 $Comp
-L +5V #PWR27
+L +5V #PWR035
 U 1 1 5533F451
 P 5150 4400
-F 0 "#PWR27" H 5150 4490 20  0001 C CNN
+F 0 "#PWR035" H 5150 4490 20  0001 C CNN
 F 1 "+5V" H 5150 4490 30  0000 C CNN
 	1    5150 4400
@@
 $EndComp
 $Comp
-L GND #PWR30
+L GND #PWR036
 U 1 1 5533F450
 P 5150 5300
-F 0 "#PWR30" H 5150 5300 30  0001 C CNN
+F 0 "#PWR036" H 5150 5300 30  0001 C CNN
 F 1 "GND" H 5150 5230 30  0001 C CNN
 	1    5150 5300

Commit message: Updated the Part number and footprints for most components
Parts:
- removed R17: 10.2K, symbol R
- added JP1: JUMPER, symbol JUMPER
- added R15: 10.2K, 0805, symbol R
- C11, C13: value 0.1uF -> 1uF; Digikey P/N 1276-1828-1-ND -> 1276-3010-1-ND; Mfg P/N CL21C151JBANNNC -> CL21F105ZBFNNNE
- C12: value 1000pF -> 1uF; Digikey P/N 1276-1828-1-ND -> 1276-3010-1-ND; Mfg P/N CL21C151JBANNNC -> CL21F105ZBFNNNE
- C14: value 0.1uF -> 1000pF; Digikey P/N 1276-1828-1-ND -> 1276-1020-1-ND; Mfg P/N CL21C151JBANNNC -> CL21B102KBANNNC
- C15: Digikey P/N 1276-1828-1-ND -> 1276-1020-1-ND; Mfg P/N CL21C151JBANNNC -> CL21B102KBANNNC
- J4: renamed from J6; value AVR-ISP-6 -> ICSP; footprint AVR-ISP-6 -> 3x2 0.1\"; Digikey P/N (none) -> 3M15451-ND; Mfg P/N (none) -> 30306-6002HB; Mouser P/N (none) -> 517-30306-6002HB
- J5: renamed from K1; value CONN_3 -> SERIAL_OUT; footprint (none) -> 3x1 0.1\"; Digikey P/N (none) -> S1012EC-40-ND; Mfg P/N (none) -> PREC040SAAN-RC
- L1: value Ferrite Bead -> 1k @ 100MHz; Digikey P/N (none) -> 587-1904-1-ND; Mfg P/N (none) -> BK2125HS102-T; Mouser P/N (none) -> 963-BK2125HS102-T
- Q1: footprint (none) -> TO-92-3; Digikey P/N (none) -> 2N3904FS-ND; Mfg P/N (none) -> 2N3904BU; Mouser P/N (none) -> 512-2N3904BU
- R13: value 57.6K -> 10.2K; footprint (none) -> 0805; Digikey P/N (none) -> P10.2KCCT-ND; Mfg P/N (none) -> ERJ-6ENF1022V; Mouser P/N (none) -> 667-ERJ-6ENF1022V
- R14, R16, R19: footprint (none) -> 0805; Digikey P/N (none) -> P10.2KCCT-ND; Mfg P/N (none) -> ERJ-6ENF1022V; Mouser P/N (none) -> 667-ERJ-6ENF1022V
- R17: renamed from R15; footprint (none) -> 0805; Digikey P/N (none) -> P1.00KCCT-ND; Mfg P/N (none) -> ERJ-6ENF1001V; Mouser P/N (none) -> 667-ERJ-6ENF1001V
- R18: value 10.2K -> 57.6K; footprint (none) -> 0805; Digikey P/N (none) -> P56.2KCCT-ND; Mfg P/N (none) -> ERJ-6ENF5622V; Mouser P/N (none) -> 667-ERJ-6ENF5622V
- U4: footprint (none) -> TQFP-32; Digikey P/N (none) -> ATMEGA64M1-15AZCT-ND; Mfg P/N (none) -> ATMEGA64M1-15AZ; Mouser P/N (none) -> 556-ATMEGA64M1-15AZ
Connections:
- net +5V: now also C13.1, JP1.1; no longer C11.2, J4.2
- net +5VA: now also C12.1; no longer C13.2
- net +BATT: now also R18.1; no longer R13.1
- net BATT_PWM: now also R13.2
- net BATT_SENSE: now also C15.1, R18.2, R19.2; no longer C12.1, R13.2, R14.1
- net GND: now also C11.2, C12.2, C13.2, C14.2; no longer C11.1, C13.1, C14.1, C15.2
- net UART_RX: now also R14.2; no longer R18.2
- net UART_TX: now also R15.1; no longer R19.1
- net nRESET: now also C14.1; no longer C15.1
- net at U4.21 (AREF): now also C11.1; no longer C14.2
- net at J4.3: now also R14.1; no longer R18.1
- net at J4.1: now also R13.1
- net at J4.4: now also R15.2; no longer R19.2
- new net: C15.2, Q1.3 (C), R19.1
- new net: J4.2, JP1.2
