File: hardware/3 Phase Inverter.sch (KiCad schematic (older format))
At the start: 21 parts, among them Q2 NTD5806N, Q3 NTD5806N, Q4 NTD5806N, Q5 NTD5806N, Q6 NTD5806N, Q7 NTD5806N, U5 LM5109, U6 LM5109, U7 LM5109

Commit message: Modified schematic to use one less op-amp and a cheaper microcontroller
Parts:
- removed R21, R22: 0.001, 2512, symbol R
- renumbered C16 to C15, C17 to C16, C18 to C17, C19 to C18, C20 to C19, C21 to C20, R20 to R16, U5 to U4, U6 to U5, U7 to U6
Connections:
- net V_CURR is gone; now on net CURR_SENSE: Q5.3 (S)
- net W_CURR is gone; now on net CURR_SENSE: Q7.3 (S)
- net U_CURR renamed CURR_SENSE
Other:
- moved on the sheet: R16

Commit message: Modified schemdatic to use a single PWM channel, similar to Atmel's app note.
Parts:
- renumbered R16 to R18, U4 to U5, U5 to U6, U6 to U7
Changed lines of the file:
@@
-EESchema Schematic File Version 2  date Fri 01 May 2015 21:46:15 MST
+EESchema Schematic File Version 2  date Wed 20 May 2015 20:05:56 MST
 LIBS:power
 LIBS:device
@@
 Sheet 4 4
 Title "3 Phase Inverter"
-Date "2 may 2015"
+Date "21 may 2015"
 Rev ""
 Comp ""
@@
 $EndComp
 $Comp
-L +BATT #PWR030
+L +BATT #PWR38
 U 1 1 553C100A
 P 8000 2150
-F 0 "#PWR030" H 8000 2100 20  0001 C CNN
+F 0 "#PWR38" H 8000 2100 20  0001 C CNN
 F 1 "+BATT" H 8000 2250 30  0000 C CNN
 	1    8000 2150
@@
 W_HI
 $Comp
-L GND #PWR031
+L GND #PWR37
 U 1 1 553C1005
 P 7350 2850
-F 0 "#PWR031" H 7350 2850 30  0001 C CNN
+F 0 "#PWR37" H 7350 2850 30  0001 C CNN
 F 1 "GND" H 7350 2780 30  0001 C CNN
 	1    7350 2850
@@
 W_OUT
 $Comp
-L IRS2301S U6
+L IRS2301S U7
 U 1 1 553C1004
 P 7750 2900
-F 0 "U6" H 7650 3100 60  0000 C CNN
+F 0 "U7" H 7650 3100 60  0000 C CNN
 F 1 "LM5109" H 7750 2700 60  0000 C CNN
 F 2 "SOIC8" H 7550 3250 60  0001 C CNN
@@
 $EndComp
 $Comp
-L IRS2301S U5
+L IRS2301S U6
 U 1 1 553C0FFD
 P 4800 2900
-F 0 "U5" H 4700 3100 60  0000 C CNN
+F 0 "U6" H 4700 3100 60  0000 C CNN
 F 1 "LM5109" H 4800 2700 60  0000 C CNN
 F 2 "SOIC8" H 4600 3250 60  0001 C CNN
@@
 V_OUT
 $Comp
-L GND #PWR032
+L GND #PWR34
 U 1 1 553C0FFC
 P 4400 2850
-F 0 "#PWR032" H 4400 2850 30  0001 C CNN
+F 0 "#PWR34" H 4400 2850 30  0001 C CNN
 F 1 "GND" H 4400 2780 30  0001 C CNN
 	1    4400 2850
@@
 V_LO
 $Comp
-L +BATT #PWR033
+L +BATT #PWR35
 U 1 1 553C0FF7
 P 5050 2150
-F 0 "#PWR033" H 5050 2100 20  0001 C CNN
+F 0 "#PWR35" H 5050 2100 20  0001 C CNN
 F 1 "+BATT" H 5050 2250 30  0000 C CNN
 	1    5050 2150
@@
 $EndComp
 $Comp
-L +BATT #PWR034
+L +BATT #PWR33
 U 1 1 553C0FD4
 P 2250 2150
-F 0 "#PWR034" H 2250 2100 20  0001 C CNN
+F 0 "#PWR33" H 2250 2100 20  0001 C CNN
 F 1 "+BATT" H 2250 2250 30  0000 C CNN
 	1    2250 2150
@@
 $EndComp
 $Comp
-L GND #PWR035
+L GND #PWR36
 U 1 1 553C0F30
 P 5700 4350
-F 0 "#PWR035" H 5700 4350 30  0001 C CNN
+F 0 "#PWR36" H 5700 4350 30  0001 C CNN
 F 1 "GND" H 5700 4280 30  0001 C CNN
 	1    5700 4350
@@
 U_HI
 $Comp
-L GND #PWR036
+L GND #PWR32
 U 1 1 5533F2AB
 P 1600 2850
-F 0 "#PWR036" H 1600 2850 30  0001 C CNN
+F 0 "#PWR32" H 1600 2850 30  0001 C CNN
 F 1 "GND" H 1600 2780 30  0001 C CNN
 	1    1600 2850
@@
 U_OUT
 $Comp
-L IRS2301S U4
+L IRS2301S U5
 U 1 1 5533F2AE
 P 2000 2900
-F 0 "U4" H 1900 3100 60  0000 C CNN
+F 0 "U5" H 1900 3100 60  0000 C CNN
 F 1 "LM5109" H 2000 2700 60  0000 C CNN
 F 2 "SOIC8" H 1800 3250 60  0001 C CNN
@@
 $EndComp
 $Comp
-L R R16
+L R R18
 U 1 1 5533F2A2
 P 5700 4050
-F 0 "R16" V 5780 4050 50  0000 C CNN
+F 0 "R18" V 5780 4050 50  0000 C CNN
 F 1 "0.001" V 5700 4050 50  0000 C CNN
 F 2 "2512" H 5700 4050 60  0001 C CNN

Commit message: Changed most parts to be through hole to simplify the initial prototype assembly
Parts:
- removed C15: 1uF, 0805, symbol C
- added C21: 1uF, symbol C
- C16, C17, C18, C19, C20: footprint 0805 -> (none); Digikey P/N 1276-3010-1-ND -> 445-8517-ND; Mfg P/N CL21F105ZBFNNNE -> FK24X7R1H105K; Mouser P/N (none) -> 810-FK24X7R1H105K
- R18: value 0.001 -> 0.01; footprint 2512 -> (none); Digikey P/N CRE2512-FZ-R001E-2CT-ND -> MPR5JB10L0-ND; Mfg P/N CRE2512-FZ-R001E-2 -> MPR5JB10L0; Mouser P/N 652-CRE2512FZR001E-2 -> (none)
Connections:
- net +BATT: now also C16.1, C18.1, C20.1; no longer C17.1, C19.1
- net GND: now also C16.2, C18.2, C20.2; no longer C17.2, C19.2
- net U_OUT: now also C17.2; no longer C16.2
- net V_OUT: now also C19.2; no longer C18.2
- net W_OUT: now also C21.2; no longer C20.2
- net at D1.2 (K), U5.8 (VB): now also C17.1; no longer C16.1
- net at D2.2 (K), U6.8 (VB): now also C19.1; no longer C18.1
- net at D3.2 (K), U7.8 (VB): now also C21.1; no longer C20.1
Changed lines of the file:
@@
-EESchema Schematic File Version 2  date Wed 20 May 2015 20:05:56 MST
+EESchema Schematic File Version 2  date Wed 20 May 2015 21:37:10 MST
 LIBS:power
 LIBS:device
@@
 Comment4 ""
 $EndDescr
+$Comp
+L C C17
+U 1 1 555D4FC4
+P 2400 2400
+F 0 "C17" H 2450 2500 50  0000 L CNN
+F 1 "1uF" H 2450 2300 50  0000 L CNN
+F 4 "FK24X7R1H105K" H 2400 2400 60  0001 C CNN "Mfg P/N"
+F 5 "445-8517-ND" H 2400 2400 60  0001 C CNN "Digikey P/N"
+F 6 "810-FK24X7R1H105K" H 2400 2400 60  0001 C CNN "Mouser P/N"
+	1    2400 2400
+	1    0    0    -1
+$EndComp
+$Comp
+L C C19
+U 1 1 555D4FC0
+P 5200 2400
+F 0 "C19" H 5250 2500 50  0000 L CNN
+F 1 "1uF" H 5250 2300 50  0000 L CNN
+F 4 "FK24X7R1H105K" H 5200 2400 60  0001 C CNN "Mfg P/N"
+F 5 "445-8517-ND" H 5200 2400 60  0001 C CNN "Digikey P/N"
+F 6 "810-FK24X7R1H105K" H 5200 2400 60  0001 C CNN "Mouser P/N"
+	1    5200 2400
+	1    0    0    -1
+$EndComp
+$Comp
+L C C21
+U 1 1 555D4FBB
+P 8150 2400
+F 0 "C21" H 8200 2500 50  0000 L CNN
+F 1 "1uF" H 8200 2300 50  0000 L CNN
+F 4 "FK24X7R1H105K" H 8150 2400 60  0001 C CNN "Mfg P/N"
+F 5 "445-8517-ND" H 8150 2400 60  0001 C CNN "Digikey P/N"
+F 6 "810-FK24X7R1H105K" H 8150 2400 60  0001 C CNN "Mouser P/N"
+	1    8150 2400
+	1    0    0    -1
+$EndComp
+$Comp
+L C C20
+U 1 1 555D4FB8
+P 7350 2550
+F 0 "C20" H 7400 2650 50  0000 L CNN
+F 1 "1uF" H 7400 2450 50  0000 L CNN
+F 4 "FK24X7R1H105K" H 7350 2550 60  0001 C CNN "Mfg P/N"
+F 5 "445-8517-ND" H 7350 2550 60  0001 C CNN "Digikey P/N"
+F 6 "810-FK24X7R1H105K" H 7350 2550 60  0001 C CNN "Mouser P/N"
+	1    7350 2550
+	-1   0    0    -1
+$EndComp
+$Comp
+L C C18
+U 1 1 555D4FB5
+P 4400 2550
+F 0 "C18" H 4450 2650 50  0000 L CNN
+F 1 "1uF" H 4450 2450 50  0000 L CNN
+F 4 "FK24X7R1H105K" H 4400 2550 60  0001 C CNN "Mfg P/N"
+F 5 "445-8517-ND" H 4400 2550 60  0001 C CNN "Digikey P/N"
+F 6 "810-FK24X7R1H105K" H 4400 2550 60  0001 C CNN "Mouser P/N"
+	1    4400 2550
+	-1   0    0    -1
+$EndComp
+$Comp
+L C C16
+U 1 1 555D4FB1
+P 1600 2550
+F 0 "C16" H 1650 2650 50  0000 L CNN
+F 1 "1uF" H 1650 2450 50  0000 L CNN
+F 4 "FK24X7R1H105K" H 1600 2550 60  0001 C CNN "Mfg P/N"
+F 5 "445-8517-ND" H 1600 2550 60  0001 C CNN "Digikey P/N"
+F 6 "810-FK24X7R1H105K" H 1600 2550 60  0001 C CNN "Mouser P/N"
+	1    1600 2550
+	-1   0    0    -1
+$EndComp
 Text HLabel 6050 3800 2    60   Output ~ 0
 CURR_SENSE
@@
 $EndComp
 $Comp
-L C C19
-U 1 1 553C2361
-P 7350 2550
-F 0 "C19" H 7400 2650 50  0000 L CNN
-F 1 "1uF" H 7400 2450 50  0000 L CNN
-F 2 "0805" H 7350 2550 60  0001 C CNN
-F 4 "CL21F105ZBFNNNE" H 7350 2550 60  0001 C CNN "Mfg P/N"
-F 5 "1276-3010-1-ND" H 7350 2550 60  0001 C CNN "Digikey P/N"
-	1    7350 2550
-	-1   0    0    -1
-$EndComp
-$Comp
-L C C17
-U 1 1 553C235E
-P 4400 2550
-F 0 "C17" H 4450 2650 50  0000 L CNN
-F 1 "1uF" H 4450 2450 50  0000 L CNN
-F 2 "0805" H 4400 2550 60  0001 C CNN
-F 4 "CL21F105ZBFNNNE" H 4400 2550 60  0001 C CNN "Mfg P/N"
-F 5 "1276-3010-1-ND" H 4400 2550 60  0001 C CNN "Digikey P/N"
-	1    4400 2550
-	-1   0    0    -1
-$EndComp
-$Comp
-L C C18
-U 1 1 553C235A
-P 5200 2400
-F 0 "C18" H 5250 2500 50  0000 L CNN
-F 1 "1uF" H 5250 2300 50  0000 L CNN
-F 2 "0805" H 5200 2400 60  0001 C CNN
-F 4 "CL21F105ZBFNNNE" H 5200 2400 60  0001 C CNN "Mfg P/N"
-F 5 "1276-3010-1-ND" H 5200 2400 60  0001 C CNN "Digikey P/N"
-	1    5200 2400
-	1    0    0    -1
-$EndComp
-$Comp
-L C C20
-U 1 1 553C2357
-P 8150 2400
-F 0 "C20" H 8200 2500 50  0000 L CNN
-F 1 "1uF" H 8200 2300 50  0000 L CNN
-F 2 "0805" H 8150 2400 60  0001 C CNN
-F 4 "CL21F105ZBFNNNE" H 8150 2400 60  0001 C CNN "Mfg P/N"
-F 5 "1276-3010-1-ND" H 8150 2400 60  0001 C CNN "Digikey P/N"
-	1    8150 2400
-	1    0    0    -1
-$EndComp
-$Comp
-L C C16
-U 1 1 553C234E
-P 2400 2400
-F 0 "C16" H 2450 2500 50  0000 L CNN
-F 1 "1uF" H 2450 2300 50  0000 L CNN
-F 2 "0805" H 2400 2400 60  0001 C CNN
-F 4 "CL21F105ZBFNNNE" H 2400 2400 60  0001 C CNN "Mfg P/N"
-F 5 "1276-3010-1-ND" H 2400 2400 60  0001 C CNN "Digikey P/N"
-	1    2400 2400
-	1    0    0    -1
-$EndComp
-$Comp
-L C C15
-U 1 1 553C2344
-P 1600 2550
-F 0 "C15" H 1650 2650 50  0000 L CNN
-F 1 "1uF" H 1650 2450 50  0000 L CNN
-F 2 "0805" H 1600 2550 60  0001 C CNN
-F 4 "CL21F105ZBFNNNE" H 1600 2550 60  0001 C CNN "Mfg P/N"
-F 5 "1276-3010-1-ND" H 1600 2550 60  0001 C CNN "Digikey P/N"
-	1    1600 2550
-	-1   0    0    -1
-$EndComp
-$Comp
-L +BATT #PWR38
+L +BATT #PWR032
 U 1 1 553C100A
 P 8000 2150
-F 0 "#PWR38" H 8000 2100 20  0001 C CNN
+F 0 "#PWR032" H 8000 2100 20  0001 C CNN
 F 1 "+BATT" H 8000 2250 30  0000 C CNN
 	1    8000 2150
@@
 W_HI
 $Comp
-L GND #PWR37
+L GND #PWR033
 U 1 1 553C1005
 P 7350 2850
-F 0 "#PWR37" H 7350 2850 30  0001 C CNN
+F 0 "#PWR033" H 7350 2850 30  0001 C CNN
 F 1 "GND" H 7350 2780 30  0001 C CNN
 	1    7350 2850
@@
 V_OUT
 $Comp
-L GND #PWR34
+L GND #PWR034
 U 1 1 553C0FFC
 P 4400 2850
-F 0 "#PWR34" H 4400 2850 30  0001 C CNN
+F 0 "#PWR034" H 4400 2850 30  0001 C CNN
 F 1 "GND" H 4400 2780 30  0001 C CNN
 	1    4400 2850
@@
 V_LO
 $Comp
-L +BATT #PWR35
+L +BATT #PWR035
 U 1 1 553C0FF7
 P 5050 2150
-F 0 "#PWR35" H 5050 2100 20  0001 C CNN
+F 0 "#PWR035" H 5050 2100 20  0001 C CNN
 F 1 "+BATT" H 5050 2250 30  0000 C CNN
 	1    5050 2150
@@
 $EndComp
 $Comp
-L +BATT #PWR33
+L +BATT #PWR036
 U 1 1 553C0FD4
 P 2250 2150
-F 0 "#PWR33" H 2250 2100 20  0001 C CNN
+F 0 "#PWR036" H 2250 2100 20  0001 C CNN
 F 1 "+BATT" H 2250 2250 30  0000 C CNN
 	1    2250 2150
@@
 $EndComp
 $Comp
-L GND #PWR36
+L GND #PWR037
 U 1 1 553C0F30
 P 5700 4350
-F 0 "#PWR36" H 5700 4350 30  0001 C CNN
+F 0 "#PWR037" H 5700 4350 30  0001 C CNN
 F 1 "GND" H 5700 4280 30  0001 C CNN
 	1    5700 4350
@@
 U_HI
 $Comp
-L GND #PWR32
+L GND #PWR038
 U 1 1 5533F2AB
 P 1600 2850
-F 0 "#PWR32" H 1600 2850 30  0001 C CNN
+F 0 "#PWR038" H 1600 2850 30  0001 C CNN
 F 1 "GND" H 1600 2780 30  0001 C CNN
 	1    1600 2850
@@
 P 5700 4050
 F 0 "R18" V 5780 4050 50  0000 C CNN
-F 1 "0.001" V 5700 4050 50  0000 C CNN
-F 2 "2512" H 5700 4050 60  0001 C CNN
-F 3 "datasheet/CRE2512.pdf" H 5700 4050 60  0001 C CNN
-F 4 "CRE2512-FZ-R001E-2" V 5700 4050 60  0001 C CNN "Mfg P/N"
-F 5 "CRE2512-FZ-R001E-2CT-ND" V 5700 4050 60  0001 C CNN "Digikey P/N"
-F 6 "652-CRE2512FZR001E-2" V 5700 4050 60  0001 C CNN "Mouser P/N"
+F 1 "0.01" V 5700 4050 50  0000 C CNN
+F 4 "MPR5JB10L0" V 5700 4050 60  0001 C CNN "Mfg P/N"
+F 5 "MPR5JB10L0-ND" V 5700 4050 60  0001 C CNN "Digikey P/N"
 	1    5700 4050
 	1    0    0    -1

Commit message: Fixed item properties and generated a BOM.
Parts:
- Q2, Q3, Q4, Q5, Q6, Q7: value NTD5806N -> NTD5865N; Digikey P/N NTD5806NT4GOSCT-ND -> NTD5865NT4GOSCT-ND; Mfg P/N NTD5806NT4G -> NTD5865NT4G; Mouser P/N 863-NTD5806NT4G -> 863-NTD5865NT4G
Changed lines of the file:
@@
-EESchema Schematic File Version 2  date Sun 14 Jun 2015 10:56:58 MST
+EESchema Schematic File Version 2  date Sun 14 Jun 2015 15:22:49 MST
 LIBS:power
 LIBS:device
@@
 $EndDescr
 $Comp
+L NTD5806N Q7
+U 1 1 557DEF8A
+P 8550 3150
+F 0 "Q7" H 8800 3300 60  0000 R CNN
+F 1 "NTD5865N" H 9200 3100 60  0000 R CNN
+F 2 "DPAK" H 8760 2870 60  0001 C CNN
+F 3 "NTD5865N-D.PDF" H 9235 2795 60  0001 C CNN
+F 4 "NTD5865NT4G" H 8550 3150 60  0001 C CNN "Mfg P/N"
+F 5 "NTD5865NT4GOSCT-ND" H 8550 3150 60  0001 C CNN "Digikey P/N"
+F 6 "863-NTD5865NT4G" H 8550 3150 60  0001 C CNN "Mouser P/N"
+	1    8550 3150
+	1    0    0    -1
+$EndComp
+$Comp
+L NTD5806N Q6
+U 1 1 557DEF88
+P 8550 2550
+F 0 "Q6" H 8800 2700 60  0000 R CNN
+F 1 "NTD5865N" H 9200 2500 60  0000 R CNN
+F 2 "DPAK" H 8760 2270 60  0001 C CNN
+F 3 "NTD5865N-D.PDF" H 9235 2195 60  0001 C CNN
+F 4 "NTD5865NT4G" H 8550 2550 60  0001 C CNN "Mfg P/N"
+F 5 "NTD5865NT4GOSCT-ND" H 8550 2550 60  0001 C CNN "Digikey P/N"
+F 6 "863-NTD5865NT4G" H 8550 2550 60  0001 C CNN "Mouser P/N"
+	1    8550 2550
+	1    0    0    -1
+$EndComp
+$Comp
+L NTD5806N Q5
+U 1 1 557DEF86
+P 5600 3150
+F 0 "Q5" H 5850 3300 60  0000 R CNN
+F 1 "NTD5865N" H 6250 3100 60  0000 R CNN
+F 2 "DPAK" H 5810 2870 60  0001 C CNN
+F 3 "NTD5865N-D.PDF" H 6285 2795 60  0001 C CNN
+F 4 "NTD5865NT4G" H 5600 3150 60  0001 C CNN "Mfg P/N"
+F 5 "NTD5865NT4GOSCT-ND" H 5600 3150 60  0001 C CNN "Digikey P/N"
+F 6 "863-NTD5865NT4G" H 5600 3150 60  0001 C CNN "Mouser P/N"
+	1    5600 3150
+	1    0    0    -1
+$EndComp
+$Comp
+L NTD5806N Q4
+U 1 1 557DEF83
+P 5600 2550
+F 0 "Q4" H 5850 2700 60  0000 R CNN
+F 1 "NTD5865N" H 6250 2500 60  0000 R CNN
+F 2 "DPAK" H 5810 2270 60  0001 C CNN
+F 3 "NTD5865N-D.PDF" H 6285 2195 60  0001 C CNN
+F 4 "NTD5865NT4G" H 5600 2550 60  0001 C CNN "Mfg P/N"
+F 5 "NTD5865NT4GOSCT-ND" H 5600 2550 60  0001 C CNN "Digikey P/N"
+F 6 "863-NTD5865NT4G" H 5600 2550 60  0001 C CNN "Mouser P/N"
+	1    5600 2550
+	1    0    0    -1
+$EndComp
+$Comp
+L NTD5806N Q3
+U 1 1 557DEF81
+P 2800 3150
+F 0 "Q3" H 3050 3300 60  0000 R CNN
+F 1 "NTD5865N" H 3450 3100 60  0000 R CNN
+F 2 "DPAK" H 3010 2870 60  0001 C CNN
+F 3 "NTD5865N-D.PDF" H 3485 2795 60  0001 C CNN
+F 4 "NTD5865NT4G" H 2800 3150 60  0001 C CNN "Mfg P/N"
+F 5 "NTD5865NT4GOSCT-ND" H 2800 3150 60  0001 C CNN "Digikey P/N"
+F 6 "863-NTD5865NT4G" H 2800 3150 60  0001 C CNN "Mouser P/N"
+	1    2800 3150
+	1    0    0    -1
+$EndComp
+$Comp
 L C C17
 U 1 1 555D4FC4
@@
 	4500 2800 4400 2800
 Connection ~ 5700 3700
-$Comp
-L NTD5806N Q7
-U 1 1 553C27F8
-P 8550 3150
-F 0 "Q7" H 8800 3300 60  0000 R CNN
-F 1 "NTD5806N" H 9200 3100 60  0000 R CNN
-F 2 "DPAK" H 8760 2870 60  0001 C CNN
-F 3 "datasheets/NTD5806N.PDF" H 9235 2795 60  0001 C CNN
-F 4 "NTD5806NT4G" H 8550 3150 60  0001 C CNN "Mfg P/N"
-F 5 "NTD5806NT4GOSCT-ND" H 8550 3150 60  0001 C CNN "Digikey P/N"
-F 6 "863-NTD5806NT4G" H 8550 3150 60  0001 C CNN "Mouser P/N"
-	1    8550 3150
-	1    0    0    -1
-$EndComp
-$Comp
-L NTD5806N Q6
-U 1 1 553C27F5
-P 8550 2550
-F 0 "Q6" H 8800 2700 60  0000 R CNN
-F 1 "NTD5806N" H 9200 2500 60  0000 R CNN
-F 2 "DPAK" H 8760 2270 60  0001 C CNN
-F 3 "datasheets/NTD5806N.PDF" H 9235 2195 60  0001 C CNN
-F 4 "NTD5806NT4G" H 8550 2550 60  0001 C CNN "Mfg P/N"
-F 5 "NTD5806NT4GOSCT-ND" H 8550 2550 60  0001 C CNN "Digikey P/N"
-F 6 "863-NTD5806NT4G" H 8550 2550 60  0001 C CNN "Mouser P/N"
-	1    8550 2550
-	1    0    0    -1
-$EndComp
-$Comp
-L NTD5806N Q5
-U 1 1 553C27F4
-P 5600 3150
-F 0 "Q5" H 5850 3300 60  0000 R CNN
-F 1 "NTD5806N" H 6250 3100 60  0000 R CNN
-F 2 "DPAK" H 5810 2870 60  0001 C CNN
-F 3 "datasheets/NTD5806N.PDF" H 6285 2795 60  0001 C CNN
-F 4 "NTD5806NT4G" H 5600 3150 60  0001 C CNN "Mfg P/N"
-F 5 "NTD5806NT4GOSCT-ND" H 5600 3150 60  0001 C CNN "Digikey P/N"
-F 6 "863-NTD5806NT4G" H 5600 3150 60  0001 C CNN "Mouser P/N"
-	1    5600 3150
-	1    0    0    -1
-$EndComp
-$Comp
-L NTD5806N Q4
-U 1 1 553C27F1
-P 5600 2550
-F 0 "Q4" H 5850 2700 60  0000 R CNN
-F 1 "NTD5806N" H 6250 2500 60  0000 R CNN
-F 2 "DPAK" H 5810 2270 60  0001 C CNN
-F 3 "datasheets/NTD5806N.PDF" H 6285 2195 60  0001 C CNN
-F 4 "NTD5806NT4G" H 5600 2550 60  0001 C CNN "Mfg P/N"
-F 5 "NTD5806NT4GOSCT-ND" H 5600 2550 60  0001 C CNN "Digikey P/N"
-F 6 "863-NTD5806NT4G" H 5600 2550 60  0001 C CNN "Mouser P/N"
-	1    5600 2550
-	1    0    0    -1
-$EndComp
-$Comp
-L NTD5806N Q3
-U 1 1 553C27EE
-P 2800 3150
-F 0 "Q3" H 3050 3300 60  0000 R CNN
-F 1 "NTD5806N" H 3450 3100 60  0000 R CNN
-F 2 "DPAK" H 3010 2870 60  0001 C CNN
-F 3 "datasheets/NTD5806N.PDF" H 3485 2795 60  0001 C CNN
-F 4 "NTD5806NT4G" H 2800 3150 60  0001 C CNN "Mfg P/N"
-F 5 "NTD5806NT4GOSCT-ND" H 2800 3150 60  0001 C CNN "Digikey P/N"
-F 6 "863-NTD5806NT4G" H 2800 3150 60  0001 C CNN "Mouser P/N"
-	1    2800 3150
-	1    0    0    -1
-$EndComp
 $Comp
 L DIODE D3
@@
 $EndComp
 $Comp
-L +BATT #PWR034
+L +BATT #PWR38
 U 1 1 553C100A
 P 8000 2150
-F 0 "#PWR034" H 8000 2100 20  0001 C CNN
+F 0 "#PWR38" H 8000 2100 20  0001 C CNN
 F 1 "+BATT" H 8000 2250 30  0000 C CNN
 	1    8000 2150
@@
 W_HI
 $Comp
-L GND #PWR035
+L GND #PWR37
 U 1 1 553C1005
 P 7350 2850
-F 0 "#PWR035" H 7350 2850 30  0001 C CNN
+F 0 "#PWR37" H 7350 2850 30  0001 C CNN
 F 1 "GND" H 7350 2780 30  0001 C CNN
 	1    7350 2850
@@
 V_OUT
 $Comp
-L GND #PWR036
+L GND #PWR34
 U 1 1 553C0FFC
 P 4400 2850
-F 0 "#PWR036" H 4400 2850 30  0001 C CNN
+F 0 "#PWR34" H 4400 2850 30  0001 C CNN
 F 1 "GND" H 4400 2780 30  0001 C CNN
 	1    4400 2850
@@
 V_LO
 $Comp
-L +BATT #PWR037
+L +BATT #PWR35
 U 1 1 553C0FF7
 P 5050 2150
-F 0 "#PWR037" H 5050 2100 20  0001 C CNN
+F 0 "#PWR35" H 5050 2100 20  0001 C CNN
 F 1 "+BATT" H 5050 2250 30  0000 C CNN
 	1    5050 2150
@@
 $EndComp
 $Comp
-L +BATT #PWR038
+L +BATT #PWR33
 U 1 1 553C0FD4
 P 2250 2150
-F 0 "#PWR038" H 2250 2100 20  0001 C CNN
+F 0 "#PWR33" H 2250 2100 20  0001 C CNN
 F 1 "+BATT" H 2250 2250 30  0000 C CNN
 	1    2250 2150
@@
 $EndComp
 $Comp
-L GND #PWR039
+L GND #PWR36
 U 1 1 553C0F30
 P 5700 4350
-F 0 "#PWR039" H 5700 4350 30  0001 C CNN
+F 0 "#PWR36" H 5700 4350 30  0001 C CNN
 F 1 "GND" H 5700 4280 30  0001 C CNN
 	1    5700 4350
@@
 P 2800 2550
 F 0 "Q2" H 3050 2700 60  0000 R CNN
-F 1 "NTD5806N" H 3450 2500 60  0000 R CNN
+F 1 "NTD5865N" H 3450 2500 60  0000 R CNN
 F 2 "DPAK" H 3010 2270 60  0001 C CNN
-F 3 "datasheets/NTD5806N.PDF" H 3485 2195 60  0001 C CNN
-F 4 "NTD5806NT4G" H 2800 2550 60  0001 C CNN "Mfg P/N"
-F 5 "NTD5806NT4GOSCT-ND" H 2800 2550 60  0001 C CNN "Digikey P/N"
-F 6 "863-NTD5806NT4G" H 2800 2550 60  0001 C CNN "Mouser P/N"
+F 3 "NTD5865N-D.PDF" H 3485 2195 60  0001 C CNN
+F 4 "NTD5865NT4G" H 2800 2550 60  0001 C CNN "Mfg P/N"
+F 5 "NTD5865NT4GOSCT-ND" H 2800 2550 60  0001 C CNN "Digikey P/N"
+F 6 "863-NTD5865NT4G" H 2800 2550 60  0001 C CNN "Mouser P/N"
 	1    2800 2550
 	1    0    0    -1
@@
 U_HI
 $Comp
-L GND #PWR040
+L GND #PWR32
 U 1 1 5533F2AB
 P 1600 2850
-F 0 "#PWR040" H 1600 2850 30  0001 C CNN
+F 0 "#PWR32" H 1600 2850 30  0001 C CNN
 F 1 "GND" H 1600 2780 30  0001 C CNN
 	1    1600 2850
